Commit message: Add files via upload

File: diff_bot_description/urdf/diff_bot.xacro (robot description, xacro)
@@ -2,6 +2,7 @@
 <robot name="diff_bot" xmlns:xacro="http://www.ros.org/wiki/xacro">
 <xacro:include filename="$(find diff_bot_description)/urdf/materials.xacro" />
-<xacro:include filename="$(find diff_bot_description)/urdf/diff_bot.trans" />
-<xacro:include filename="$(find diff_bot_description)/urdf/diff_bot.gazebo" />
+<!--<xacro:include filename="$(find diff_bot_description)/urdf/diff_bot.trans" /> -->
+<!--<xacro:include filename="$(find diff_bot_description)/urdf/diff_bot.gazebo" /> -->
+<link name="base_footprint"/>
 <link name="base_link">
   <inertial>
@@ -64,5 +65,10 @@
   </collision>
 </link>
-<joint name="Revolute 1" type="continuous">
+<joint name="fixed" type="fixed">
+  <orgin xyz="0 0 0" rpy="0 0 0"/>
+  <parent link="base_footprint"/>
+  <child link="base_link"/>
+</joint>
+<joint name="right_wheel_joint" type="continuous">
   <origin xyz="0.2 0.24 0.035" rpy="0 0 0"/>
   <parent link="base_link"/>
@@ -70,5 +76,5 @@
   <axis xyz="0.0 1.0 0.0"/>
 </joint>
-<joint name="Revolute 2" type="continuous">
+<joint name="left_wheel_joint" type="continuous">
   <origin xyz="0.2 -0.24 0.035" rpy="0 0 0"/>
   <parent link="base_link"/>
@@ -76,3 +82,29 @@
   <axis xyz="0.0 1.0 0.0"/>
 </joint>
+<ros2_control name="GazeboSystem" type="system">
+  <hardware>
+    <plugin>gazebo_ros2_control/GazeboSystem</plugin>
+  </hardware>
+  <joint name="right_wheel_joint">
+    <command_interface name="velocity">
+      <param name="min">-10</param>
+      <param name="max">10</param>
+    </command_interface>
+    <state_interface name="position"/>
+    <state_interface name="velocity"/>
+  </joint>
+    <joint name="right_wheel_joint">
+    <command_interface name="velocity">
+      <param name="min">-10</param>
+      <param name="max">10</param>
+    </command_interface>
+    <state_interface name="position"/>
+    <state_interface name="velocity"/>
+  </joint>
+</ros2_control>
+<gazebo>
+  <plugin filename="libgazebo_ros2_control.so" name="gazebo_ros2_control">
+    <parameters>$(find diff_bot_description)/config/my_controller.yaml</parameters>
+  </plugin>
+</gazebo>
 </robot>

Commit message: Add files via upload

File: diff_bot_description/urdf/diff_bot.xacro (robot description, xacro)
@@ -66,5 +66,5 @@
 </link>
 <joint name="fixed" type="fixed">
-  <orgin xyz="0 0 0" rpy="0 0 0"/>
+  <origin xyz="0 0 0" rpy="0 0 0"/>
   <parent link="base_footprint"/>
   <child link="base_link"/>
@@ -94,5 +94,5 @@
     <state_interface name="velocity"/>
   </joint>
-    <joint name="right_wheel_joint">
+    <joint name="left_wheel_joint">
     <command_interface name="velocity">
       <param name="min">-10</param>

Commit message: Add files via upload

File: diff_bot_description/urdf/diff_bot.xacro (robot description, xacro)
@@ -86,5 +86,5 @@
     <plugin>gazebo_ros2_control/GazeboSystem</plugin>
   </hardware>
-  <joint name="right_wheel_joint">
+  <joint name="left_wheel_joint">
     <command_interface name="velocity">
       <param name="min">-10</param>
@@ -94,5 +94,5 @@
     <state_interface name="velocity"/>
   </joint>
-    <joint name="left_wheel_joint">
+    <joint name="right_wheel_joint">
     <command_interface name="velocity">
       <param name="min">-10</param>

Commit message: Add files via upload

File: diff_bot_description/urdf/diff_bot.xacro (robot description, xacro)
@@ -4,5 +4,5 @@
 <!--<xacro:include filename="$(find diff_bot_description)/urdf/diff_bot.trans" /> -->
 <!--<xacro:include filename="$(find diff_bot_description)/urdf/diff_bot.gazebo" /> -->
-<link name="base_footprint"/>
+<!--<link name="base_footprint"/>-->
 <link name="base_link">
   <inertial>
@@ -65,9 +65,9 @@
   </collision>
 </link>
-<joint name="fixed" type="fixed">
+<!--<joint name="fixed" type="fixed">
   <origin xyz="0 0 0" rpy="0 0 0"/>
   <parent link="base_footprint"/>
   <child link="base_link"/>
-</joint>
+</joint> -->
 <joint name="right_wheel_joint" type="continuous">
   <origin xyz="0.2 0.24 0.035" rpy="0 0 0"/>

Commit message: updated with nav2_stack

File: diff_bot_description/urdf/diff_bot.xacro (robot description, xacro)
@@ -3,6 +3,6 @@
 <xacro:include filename="$(find diff_bot_description)/urdf/materials.xacro" />
 <!--<xacro:include filename="$(find diff_bot_description)/urdf/diff_bot.trans" /> -->
-<!--<xacro:include filename="$(find diff_bot_description)/urdf/diff_bot.gazebo" /> -->
-<link name="base_footprint"/>
+<xacro:include filename="$(find diff_bot_description)/urdf/diff_bot.gazebo" />
+<!--<link name="base_footprint"/>-->
 <link name="base_link">
   <inertial>
@@ -65,9 +65,9 @@
   </collision>
 </link>
-<joint name="fixed" type="fixed">
+<!--<joint name="fixed" type="fixed">
   <origin xyz="0 0 0" rpy="0 0 0"/>
   <parent link="base_footprint"/>
   <child link="base_link"/>
-</joint>
+</joint> -->
 <joint name="right_wheel_joint" type="continuous">
   <origin xyz="0.2 0.24 0.035" rpy="0 0 0"/>
@@ -88,10 +88,10 @@
   <joint name="left_wheel_joint">
     <command_interface name="velocity"/>
-    <!--<state_interface name="position"/>-->
+    <state_interface name="position"/>
     <state_interface name="velocity"/>
   </joint>
     <joint name="right_wheel_joint">
     <command_interface name="velocity"/>
-    <!--<state_interface name="position"/>-->
+    <state_interface name="position"/>
     <state_interface name="velocity"/>
   </joint>
@@ -102,3 +102,109 @@
   </plugin>
 </gazebo>
+ <!--setting up LIDAR sensor  -->
+<link name="lidar_link">
+  <inertial>
+    <origin xyz="0 0 0" rpy="0 0 0"/>
+    <mass value="0.125"/>
+    <inertia ixx="0.001"  ixy="0"  ixz="0" iyy="0.001" iyz="0" izz="0.001" />
+  </inertial>
+  <collision>
+    <origin xyz="0 0 0" rpy="0 0 0"/>
+    <geometry>
+       <cylinder radius="0.0508" length="0.055"/>
+    </geometry>
+  </collision>
+  <visual>
+    <origin xyz="0 0 0" rpy="0 0 0"/>
+    <geometry>
+       <cylinder radius="0.0508" length="0.055"/>
+    </geometry>
+  </visual>
+</link>
+<joint name="lidar_joint" type="fixed">
+  <parent link="base_link"/>
+  <child link="lidar_link"/>
+  <origin xyz="0 0 0.15" rpy="0 0 0"/>
+</joint>
+<gazebo reference="lidar_link">
+  <sensor name="lidar" type="ray">
+    <always_on>true</always_on>
+    <visualize>true</visualize>
+    <update_rate>5</update_rate>
+    <ray>
+      <scan>
+        <horizontal>
+          <samples>360</samples>
+          <resolution>1.000000</resolution>
+          <min_angle>0.000000</min_angle>
+          <max_angle>6.280000</max_angle>
+        </horizontal>
+      </scan>
+      <range>
+        <min>0.120000</min>
+        <max>3.5</max>
+        <resolution>0.015000</resolution>
+      </range>
+      <noise>
+        <type>gaussian</type>
+        <mean>0.0</mean>
+        <stddev>0.01</stddev>
+      </noise>
+    </ray>
+    <plugin name="scan" filename="libgazebo_ros_ray_sensor.so">
+      <ros>
+        <remapping>~/out:=laser_scan</remapping>
+      </ros>
+      <output_type>sensor_msgs/LaserScan</output_type>
+      <frame_name>lidar_link</frame_name>
+    </plugin>
+  </sensor>
+</gazebo>
+<!--       setting up IMU                 -->
+<link name="imu_sensor_link">
+  <collision>
+    <origin xyz="0 0 0" rpy="0 0 0"/>
+    <geometry>
+        <box size="0.02 0.02 0.02"/>
+    </geometry>
+  </collision>
+  <visual>
+    <origin xyz="0 0 0" rpy="0 0 0"/>
+      <geometry>
+        <box size="0.02 0.02 0.02"/>
+      </geometry>
+    <material name="silver"/>
+  </visual>
+    <inertial>
+      <mass value="0.001" />
+      <origin xyz="0 0 0" rpy="0 0 0"/>
+      <inertia ixx="0.00000015" ixy="0" ixz="0" iyy="0.00000015" iyz="0" izz="0.00000015" />
+    </inertial>
+</link>
+<joint name="imu_sensor_joint" type="fixed">
+  <parent link="base_link"/>
+  <child link="imu_sensor_link"/>
+  <origin xyz="0.26 0.0 0.07" rpy="0 0 0"/>
+</joint>
+<gazebo reference="imu_sensor_link">
+  <gravity>true</gravity>
+  <sensor name='imu_sensor' type='imu'>
+    <always_on>1</always_on>
+    <update_rate>100</update_rate>
+    <visualize>1</visualize>
+    <topic>__default_topic__</topic>
+    <plugin name='imu' filename='libgazebo_ros_imu_sensor.so'>
+      <topicName>imu</topicName>
+      <ros>
+        <remapping>~/out:=imu_data</remapping>
+      </ros>
+      <bodyName>imu_sensor_link</bodyName>
+      <updateRateHZ>100.0</updateRateHZ>
+      <gaussianNoise>0.0</gaussianNoise>
+      <xyzOffset>0 0 0</xyzOffset>
+      <rpyOffset>0 0 0</rpyOffset>
+    </plugin>
+    <pose>0 0 0 0 0 0</pose>
+  </sensor>
+</gazebo>
 </robot>

Commit message: updated-DEC

File: diff_bot_description/urdf/diff_bot.xacro (robot description, xacro)
@@ -2,7 +2,6 @@
 <robot name="diff_bot" xmlns:xacro="http://www.ros.org/wiki/xacro">
 <xacro:include filename="$(find diff_bot_description)/urdf/materials.xacro" />
-<!--<xacro:include filename="$(find diff_bot_description)/urdf/diff_bot.trans" /> -->
-<!--<xacro:include filename="$(find diff_bot_description)/urdf/diff_bot.gazebo" /> -->
-<link name="base_footprint"/>
+<xacro:include filename="$(find diff_bot_description)/urdf/diff_bot.ros2_control.xacro" />
+<xacro:include filename="$(find diff_bot_description)/urdf/diff_bot.gazebo" />
 <link name="base_link">
   <inertial>
@@ -65,9 +64,4 @@
   </collision>
 </link>
-<joint name="fixed" type="fixed">
-  <origin xyz="0 0 0" rpy="0 0 0"/>
-  <parent link="base_footprint"/>
-  <child link="base_link"/>
-</joint>
 <joint name="right_wheel_joint" type="continuous">
   <origin xyz="0.2 0.24 0.035" rpy="0 0 0"/>
@@ -82,23 +76,52 @@
   <axis xyz="0.0 1.0 0.0"/>
 </joint>
-<ros2_control name="GazeboSystem" type="system">
-  <hardware>
-    <plugin>gazebo_ros2_control/GazeboSystem</plugin>
-  </hardware>
-  <joint name="left_wheel_joint">
-    <command_interface name="velocity"/>
-    <!--<state_interface name="position"/>-->
-    <state_interface name="velocity"/>
-  </joint>
-    <joint name="right_wheel_joint">
-    <command_interface name="velocity"/>
-    <!--<state_interface name="position"/>-->
-    <state_interface name="velocity"/>
-  </joint>
-</ros2_control>
-<gazebo>
-  <plugin filename="libgazebo_ros2_control.so" name="gazebo_ros2_control">
-    <parameters>$(find diff_bot_description)/config/robot_controller.yaml</parameters>
-  </plugin>
-</gazebo>
+<link name="lidar_link">
+  <inertial>
+    <origin xyz="0 0 0" rpy="0 0 0"/>
+    <mass value="0.125"/>
+    <inertia ixx="0.001"  ixy="0"  ixz="0" iyy="0.001" iyz="0" izz="0.001" />
+  </inertial>
+  <collision>
+    <origin xyz="0 0 0" rpy="0 0 0"/>
+    <geometry>
+       <cylinder radius="0.0508" length="0.055"/>
+    </geometry>
+  </collision>
+  <visual>
+    <origin xyz="0 0 0" rpy="0 0 0"/>
+    <geometry>
+       <cylinder radius="0.0508" length="0.055"/>
+    </geometry>
+  </visual>
+</link>
+<joint name="lidar_joint" type="fixed">
+  <parent link="base_link"/>
+  <child link="lidar_link"/>
+  <origin xyz="0 0 0.15" rpy="0 0 0"/>
+</joint>
+<link name="imu_link">
+  <collision>
+    <origin xyz="0 0 0" rpy="0 0 0"/>
+    <geometry>
+        <box size="0.02 0.02 0.02"/>
+    </geometry>
+  </collision>
+  <visual>
+    <origin xyz="0 0 0" rpy="0 0 0"/>
+      <geometry>
+        <box size="0.02 0.02 0.02"/>
+      </geometry>
+    <material name="silver"/>
+  </visual>
+    <inertial>
+      <mass value="0.001" />
+      <origin xyz="0 0 0" rpy="0 0 0"/>
+      <inertia ixx="0.00000015" ixy="0" ixz="0" iyy="0.00000015" iyz="0" izz="0.00000015" />
+    </inertial>
+</link>
+<joint name="imu_sensor_joint" type="fixed">
+  <parent link="base_link"/>
+  <child link="imu_link"/>
+  <origin xyz="0.0 0.0 0.0" rpy="0 0 0"/>
+</joint>
 </robot>
